Commit message: debug seesaw environment

File: resources/objects/seesaw.urdf (robot description, URDF)
Before this commit: robot sheep, 5 links, 4 joints
Links:
- link base: geometry collision box size=1 1.5 0.03; visual box size=1 1.5 0.03
- link seesaw: geometry collision box size=4.123 1.5 0.03; visual box size=4.123 1.5 0.03

Commit message: update seesaw env

File: resources/objects/seesaw.urdf (robot description, URDF)
Before this commit: robot sheep, 5 links, 4 joints
Links:
- link seesaw: geometry collision box size=4.123 1.5 0.01; visual box size=4.123 1.5 0.01
