Commit message: debug pushbox

File: resources/objects/box.urdf (robot description, URDF)
Before this commit: robot box, 1 links, 0 joints
Links:
- link box: mass 6 -> 3

Commit message: make box larger

File: resources/objects/box.urdf (robot description, URDF)
Before this commit: robot box, 1 links, 0 joints
Links:
- link box: mass 3 -> 6; geometry collision box size=0.5 1.5 0.5; visual box size=0.5 1.5 0.5

Commit message: randomize target position

File: resources/objects/box.urdf (robot description, URDF)
Before this commit: robot box, 1 links, 0 joints
Links:
- link box: geometry collision box size=1.0 1.0 0.8; visual box size=1.0 1.0 0.8

Commit message: wide box

File: resources/objects/box.urdf (robot description, URDF)
Before this commit: robot box, 1 links, 0 joints
Links:
- link box: geometry collision box size=1.0 3.0 0.8; visual box size=1.0 3.0 0.8
